Commit message: Update mobile_robot file to match with meshes

File: ros_packages/robots_description/urdf/mobile_robot.urdf (robot description, URDF)
Before this commit: robot mobile_robot, 9 links, 8 joints
Links:
- link base_link: geometry collision box size=0.3 0.4 0.025; visual mesh filename=package://robots_description/meshes/undercarriage.dae
- link hub_bl: geometry collision box size=0.05 0.05 0.065; visual mesh filename=package://robots_description/meshes/hub.dae
- link hub_br: geometry collision box size=0.05 0.05 0.065; visual mesh filename=package://robots_description/meshes/hub.dae
- link hub_hl: geometry collision box size=0.05 0.05 0.065; visual mesh filename=package://robots_description/meshes/hub.dae
- link hub_hr: geometry collision box size=0.05 0.05 0.065; visual mesh filename=package://robots_description/meshes/hub.dae
- link wheel_bl: geometry collision mesh filename=package://robots_description/meshes/wheel_collision.dae; visual mesh filename=package://robots_description/meshes/wheel.dae
- link wheel_br: geometry collision mesh filename=package://robots_description/meshes/wheel_collision.dae; visual mesh filename=package://robots_description/meshes/wheel.dae
- link wheel_hl: geometry collision mesh filename=package://robots_description/meshes/wheel_collision.dae; visual mesh filename=package://robots_description/meshes/wheel.dae
- link wheel_hr: geometry collision mesh filename=package://robots_description/meshes/wheel_collision.dae; visual mesh filename=package://robots_description/meshes/wheel.dae

File: ros_packages/robots_description/urdf/mobile_robot_macro.xacro (robot description, xacro)
@@ -4,8 +4,8 @@
 	  <link name="${prefix}base_link">
 	    <visual>
-	      <!--undercarriage001-->
-	      <origin rpy="0.0 -0.0 -1.570796326794897" xyz="0.0 0.0 0.0"/>
-	      <geometry>
-		<mesh filename="package://robots_description/meshes/undercarriage001.dae"/>
+	      <!--undercarriage-->
+	      <origin rpy="0.0 -0.0 -1.570796326794897" xyz="0.0 0.0 0.0"/>
+	      <geometry>
+		<mesh filename="package://robots_description/meshes/undercarriage.dae"/>
 	      </geometry>
 	    </visual>
@@ -24,8 +24,8 @@
 	  <link name="${prefix}hub_hr">
 	    <visual>
-	      <!--hub001-->
-	      <origin rpy="0.0 -0.0 -1.570796326794897" xyz="0.0 0.0 0.0"/>
-	      <geometry>
-		<mesh filename="package://robots_description/meshes/hub001.dae"/>
+	      <!--hub-->
+	      <origin rpy="0.0 -0.0 -1.570796326794897" xyz="0.0 0.0 0.0"/>
+	      <geometry>
+		<mesh filename="package://robots_description/meshes/hub.dae"/>
 	      </geometry>
 	    </visual>
@@ -44,8 +44,8 @@
 	  <link name="${prefix}hub_hl">
 	    <visual>
-	      <!--hub001-->
-	      <origin rpy="0.0 -0.0 -1.570796326794897" xyz="0.0 0.0 0.0"/>
-	      <geometry>
-		<mesh filename="package://robots_description/meshes/hub001.dae"/>
+	      <!--hub-->
+	      <origin rpy="0.0 -0.0 -1.570796326794897" xyz="0.0 0.0 0.0"/>
+	      <geometry>
+		<mesh filename="package://robots_description/meshes/hub.dae"/>
 	      </geometry>
 	    </visual>
@@ -64,8 +64,8 @@
 	  <link name="${prefix}hub_br">
 	    <visual>
-	      <!--hub001-->
-	      <origin rpy="0.0 -0.0 -1.570796326794897" xyz="0.0 0.0 0.0"/>
-	      <geometry>
-		<mesh filename="package://robots_description/meshes/hub001.dae"/>
+	      <!--hub-->
+	      <origin rpy="0.0 -0.0 -1.570796326794897" xyz="0.0 0.0 0.0"/>
+	      <geometry>
+		<mesh filename="package://robots_description/meshes/hub.dae"/>
 	      </geometry>
 	    </visual>
@@ -84,8 +84,8 @@
 	  <link name="${prefix}hub_bl">
 	    <visual>
-	      <!--hub001-->
-	      <origin rpy="0.0 -0.0 -1.570796326794897" xyz="0.0 0.0 0.0"/>
-	      <geometry>
-		<mesh filename="package://robots_description/meshes/hub001.dae"/>
+	      <!--hub-->
+	      <origin rpy="0.0 -0.0 -1.570796326794897" xyz="0.0 0.0 0.0"/>
+	      <geometry>
+		<mesh filename="package://robots_description/meshes/hub.dae"/>
 	      </geometry>
 	    </visual>
@@ -104,15 +104,15 @@
 	  <link name="${prefix}wheel_hr">
 	    <visual>
-	      <!--Body002-->
-	      <origin rpy="3.141592653589793 -0.0 -1.570796326794897" xyz="0.0 0.0 0.01"/>
-	      <geometry>
-		<mesh filename="package://robots_description/meshes/Body002.dae"/>
-	      </geometry>
-	    </visual>
-	    <collision>
-	      <!--Body003-->
-	      <origin rpy="3.141592653589793 -0.0 -1.570796326794897" xyz="0.0 0.0 0.01"/>
-	      <geometry>
-		<mesh filename="package://robots_description/meshes/Body003.dae"/>
+	      <!--wheel-->
+	      <origin rpy="3.141592653589793 -0.0 -1.570796326794897" xyz="0.0 0.0 0.01"/>
+	      <geometry>
+		<mesh filename="package://robots_description/meshes/wheel.dae"/>
+	      </geometry>
+	    </visual>
+	    <collision>
+	      <!--wheel_collision-->
+	      <origin rpy="3.141592653589793 -0.0 -1.570796326794897" xyz="0.0 0.0 0.01"/>
+	      <geometry>
+		<mesh filename="package://robots_description/meshes/wheel_collision.dae"/>
 	      </geometry>
 	    </collision>
@@ -125,15 +125,15 @@
 	  <link name="${prefix}wheel_hl">
 	    <visual>
-	      <!--Body002-->
-	      <origin rpy="3.141592653589793 -0.0 -1.570796326794897" xyz="0.0 0.0 0.01"/>
-	      <geometry>
-		<mesh filename="package://robots_description/meshes/Body002.dae"/>
-	      </geometry>
-	    </visual>
-	    <collision>
-	      <!--Body003-->
-	      <origin rpy="3.141592653589793 -0.0 -1.570796326794897" xyz="0.0 0.0 0.01"/>
-	      <geometry>
-		<mesh filename="package://robots_description/meshes/Body003.dae"/>
+	      <!--wheel-->
+	      <origin rpy="3.141592653589793 -0.0 -1.570796326794897" xyz="0.0 0.0 0.01"/>
+	      <geometry>
+		<mesh filename="package://robots_description/meshes/wheel.dae"/>
+	      </geometry>
+	    </visual>
+	    <collision>
+	      <!--wheel_collision-->
+	      <origin rpy="3.141592653589793 -0.0 -1.570796326794897" xyz="0.0 0.0 0.01"/>
+	      <geometry>
+		<mesh filename="package://robots_description/meshes/wheel_collision.dae"/>
 	      </geometry>
 	    </collision>
@@ -146,15 +146,15 @@
 	  <link name="${prefix}wheel_br">
 	    <visual>
-	      <!--Body002-->
-	      <origin rpy="3.141592653589793 -0.0 -1.570796326794897" xyz="0.0 0.0 0.01"/>
-	      <geometry>
-		<mesh filename="package://robots_description/meshes/Body002.dae"/>
-	      </geometry>
-	    </visual>
-	    <collision>
-	      <!--Body003-->
-	      <origin rpy="3.141592653589793 -0.0 -1.570796326794897" xyz="0.0 0.0 0.01"/>
-	      <geometry>
-		<mesh filename="package://robots_description/meshes/Body003.dae"/>
+	      <!--wheel-->
+	      <origin rpy="3.141592653589793 -0.0 -1.570796326794897" xyz="0.0 0.0 0.01"/>
+	      <geometry>
+		<mesh filename="package://robots_description/meshes/wheel.dae"/>
+	      </geometry>
+	    </visual>
+	    <collision>
+	      <!--wheel_collision-->
+	      <origin rpy="3.141592653589793 -0.0 -1.570796326794897" xyz="0.0 0.0 0.01"/>
+	      <geometry>
+		<mesh filename="package://robots_description/meshes/wheel_collision.dae"/>
 	      </geometry>
 	    </collision>
@@ -167,15 +167,15 @@
 	  <link name="${prefix}wheel_bl">
 	    <visual>
-	      <!--Body002-->
-	      <origin rpy="3.141592653589793 -0.0 -1.570796326794897" xyz="0.0 0.0 0.01"/>
-	      <geometry>
-		<mesh filename="package://robots_description/meshes/Body002.dae"/>
-	      </geometry>
-	    </visual>
-	    <collision>
-	      <!--Body003-->
-	      <origin rpy="3.141592653589793 -0.0 -1.570796326794897" xyz="0.0 0.0 0.01"/>
-	      <geometry>
-		<mesh filename="package://robots_description/meshes/Body003.dae"/>
+	      <!--wheel-->
+	      <origin rpy="3.141592653589793 -0.0 -1.570796326794897" xyz="0.0 0.0 0.01"/>
+	      <geometry>
+		<mesh filename="package://robots_description/meshes/wheel.dae"/>
+	      </geometry>
+	    </visual>
+	    <collision>
+	      <!--wheel_collision-->
+	      <origin rpy="3.141592653589793 -0.0 -1.570796326794897" xyz="0.0 0.0 0.01"/>
+	      <geometry>
+		<mesh filename="package://robots_description/meshes/wheel_collision.dae"/>
 	      </geometry>
 	    </collision>
